File: Hardware/RGB Matrix.brd (EAGLE design)
At the start: 55.9 x 58.4 mm, 49 parts, among them IC1 74LS595D, IC2 74LS595D, IC3 AVR-MEGA8-AI, IC4 74LS595D, U2 AVR_SPI_PRG_6PTH, U3 16 MHz

Commit message: Updated revision to symbol
Parts:
- added U$2: REVISION, SparkFun-Aesthetics:REVISION
Other:
- board text added: "R. Owens"
- board text added: "T. Klopfenstein"
- board text removed: "R. Owens, Revision by: T. Klopfenstein"
